Commit message: added args to setup world_joint geometry allowing to define the position of the base_link relative to the world frame

File: ur_robot_server/urdf/ur.xacro (robot description, xacro)
@@ -30,4 +30,10 @@
   <xacro:arg name="kinematics_params" default=""/>
   <xacro:arg name="visual_params" default=""/>
+  <xacro:arg name="x" default="0.0"/>
+  <xacro:arg name="y" default="0.0"/>
+  <xacro:arg name="z" default="0.1"/>
+  <xacro:arg name="roll" default="0.0"/>
+  <xacro:arg name="pitch" default="0.0"/>
+  <xacro:arg name="yaw" default="0.0"/>
   <!--
     legal values:
@@ -65,5 +71,5 @@
     <parent link="world"/>
     <child link="base_link"/>
-    <origin xyz="0 0 0" rpy="0 0 0"/>
+    <origin xyz="$(arg x) $(arg y) $(arg z)" rpy="$(arg roll) $(arg pitch) $(arg yaw)" />
   </joint>
 </robot>

Commit message: integrate simulated gazebo camera

File: ur_robot_server/urdf/ur.xacro (robot description, xacro)
@@ -48,4 +48,12 @@
   <xacro:arg name="safety_pos_margin" default="0.15"/>
   <xacro:arg name="safety_k_position" default="20"/>
+  <!-- rgbd camera arguments -->
+  <xacro:arg name="camera1_gazebo" default="False"/>
+  <xacro:arg name="camera1_link_x" default="0.0"/>
+  <xacro:arg name="camera1_link_y" default="0.0"/>
+  <xacro:arg name="camera1_link_z" default="0.0"/>
+  <xacro:arg name="camera1_link_roll" default="0.0"/>
+  <xacro:arg name="camera1_link_pitch" default="0.0"/>
+  <xacro:arg name="camera1_link_yaw" default="0.0"/>
   <!-- Instantiate the Gazebo robot and pass it all the required arguments. -->
   <xacro:ur_robot_gazebo
@@ -73,3 +81,14 @@
     <origin xyz="$(arg x) $(arg y) $(arg z)" rpy="$(arg roll) $(arg pitch) $(arg yaw)" />
   </joint>
+  <!-- simulated rgbd camera include -->
+  <xacro:if value="$(arg camera1_gazebo)">
+    <xacro:include filename="$(find scene_perception)/urdf/rgbd_camera_macro.xacro"/>
+    <xacro:rgbd_camera_gazebo camera_name="camera1"/>
+    <joint name="camera1_joint" type="fixed">
+      <parent link="world"/>
+      <child link="camera1_link"/>
+      <origin xyz="$(arg camera1_link_x) $(arg camera1_link_y) $(arg camera1_link_z)"
+        rpy="$(arg camera1_link_roll) $(arg camera1_link_pitch) $(arg camera1_link_yaw)" />
+    </joint>
+  </xacro:if>
 </robot>
